Commit message: kniect added successfully

File: nag_raj_description/urdf/nag_raj.xacro (robot description, xacro)
@@ -1,157 +1,193 @@
-<?xml version="1.0" ?>
+<?xml version="1.0"?>
 <robot name="nag_raj" xmlns:xacro="http://www.ros.org/wiki/xacro">
-<xacro:include filename="$(find nag_raj_description)/urdf/materials.xacro" />
-<xacro:include filename="$(find nag_raj_description)/urdf/nag_raj.trans" />
-<xacro:include filename="$(find nag_raj_description)/urdf/nag_raj.gazebo" />
-<link name="base_link">
-  <inertial>
-    <origin xyz="-0.0006379139080881657 -0.01809373210164651 0.030365961397063188" rpy="0 0 0"/>
-    <mass value="12.627463545285623"/>
-    <inertia ixx="0.031143" iyy="0.030205" izz="0.052676" ixy="-0.000405" iyz="0.000267" ixz="-7e-05"/>
-  </inertial>
-  <visual>
-    <origin xyz="0 0 0" rpy="0 0 0"/>
-    <geometry>
-      <mesh filename="package://nag_raj_description/meshes/base_link.stl" scale="0.001 0.001 0.001"/>
-    </geometry>
-    <material name="silver"/>
-  </visual>
-  <collision>
-    <origin xyz="0 0 0" rpy="0 0 0"/>
-    <geometry>
-      <mesh filename="package://nag_raj_description/meshes/base_link.stl" scale="0.001 0.001 0.001"/>
-    </geometry>
-  </collision>
-</link>
-<link name="sh_joint_1">
-  <inertial>
-    <origin xyz="-0.0011960436685277943 0.0013481214024438706 0.07489085893279906" rpy="0 0 0"/>
-    <mass value="29.69776516715868"/>
-    <inertia ixx="0.099358" iyy="0.132845" izz="0.135929" ixy="0.016934" iyz="3.3e-05" ixz="-0.000187"/>
-  </inertial>
-  <visual>
-    <origin xyz="0.001039 0.018393 -0.067132" rpy="0 0 0"/>
-    <geometry>
-      <mesh filename="package://nag_raj_description/meshes/sh_joint_1.stl" scale="0.001 0.001 0.001"/>
-    </geometry>
-    <material name="silver"/>
-  </visual>
-  <collision>
-    <origin xyz="0.001039 0.018393 -0.067132" rpy="0 0 0"/>
-    <geometry>
-      <mesh filename="package://nag_raj_description/meshes/sh_joint_1.stl" scale="0.001 0.001 0.001"/>
-    </geometry>
-  </collision>
-</link>
-<link name="shoulder_1">
-  <inertial>
-    <origin xyz="0.007821760472450007 0.2778220009300011 0.03125519386875361" rpy="0 0 0"/>
-    <mass value="89.21154259038471"/>
-    <inertia ixx="4.45732" iyy="1.046726" izz="5.155255" ixy="-1.710485" iyz="-0.557906" ixz="-0.232136"/>
-  </inertial>
-  <visual>
-    <origin xyz="0.093573 -0.021145 -0.146342" rpy="0 0 0"/>
-    <geometry>
-      <mesh filename="package://nag_raj_description/meshes/shoulder_1.stl" scale="0.001 0.001 0.001"/>
-    </geometry>
-    <material name="silver"/>
-  </visual>
-  <collision>
-    <origin xyz="0.093573 -0.021145 -0.146342" rpy="0 0 0"/>
-    <geometry>
-      <mesh filename="package://nag_raj_description/meshes/shoulder_1.stl" scale="0.001 0.001 0.001"/>
-    </geometry>
-  </collision>
-</link>
-<link name="elbow1_1">
-  <inertial>
-    <origin xyz="0.012063915743866088 -0.08935136984735537 0.01819736606366848" rpy="0 0 0"/>
-    <mass value="12.818945015869657"/>
-    <inertia ixx="0.078237" iyy="0.022075" izz="0.079476" ixy="-0.01847" iyz="0.01453" ixz="0.004333"/>
-  </inertial>
-  <visual>
-    <origin xyz="-0.129699 -0.612043 -0.224144" rpy="0 0 0"/>
-    <geometry>
-      <mesh filename="package://nag_raj_description/meshes/elbow1_1.stl" scale="0.001 0.001 0.001"/>
-    </geometry>
-    <material name="silver"/>
-  </visual>
-  <collision>
-    <origin xyz="-0.129699 -0.612043 -0.224144" rpy="0 0 0"/>
-    <geometry>
-      <mesh filename="package://nag_raj_description/meshes/elbow1_1.stl" scale="0.001 0.001 0.001"/>
-    </geometry>
-  </collision>
-</link>
-<link name="elbow2_1">
-  <inertial>
-    <origin xyz="-0.06172372576999953 -0.1471990074107003 0.039999758385676654" rpy="0 0 0"/>
-    <mass value="14.074723611721877"/>
-    <inertia ixx="0.09516" iyy="0.034386" izz="0.105805" ixy="-0.030922" iyz="0.020824" ixz="0.008622"/>
-  </inertial>
-  <visual>
-    <origin xyz="-0.092673 -0.388118 -0.275308" rpy="0 0 0"/>
-    <geometry>
-      <mesh filename="package://nag_raj_description/meshes/elbow2_1.stl" scale="0.001 0.001 0.001"/>
-    </geometry>
-    <material name="silver"/>
-  </visual>
-  <collision>
-    <origin xyz="-0.092673 -0.388118 -0.275308" rpy="0 0 0"/>
-    <geometry>
-      <mesh filename="package://nag_raj_description/meshes/elbow2_1.stl" scale="0.001 0.001 0.001"/>
-    </geometry>
-  </collision>
-</link>
-<link name="wrist_1">
-  <inertial>
-    <origin xyz="-0.05432751125838708 0.017695228247820827 -0.0008664628207630809" rpy="0 0 0"/>
-    <mass value="5.82092033198201"/>
-    <inertia ixx="0.006574" iyy="0.008357" izz="0.009234" ixy="0.000912" iyz="0.000122" ixz="-5e-05"/>
-  </inertial>
-  <visual>
-    <origin xyz="0.055527 -0.184746 -0.334878" rpy="0 0 0"/>
-    <geometry>
-      <mesh filename="package://nag_raj_description/meshes/wrist_1.stl" scale="0.001 0.001 0.001"/>
-    </geometry>
-    <material name="silver"/>
-  </visual>
-  <collision>
-    <origin xyz="0.055527 -0.184746 -0.334878" rpy="0 0 0"/>
-    <geometry>
-      <mesh filename="package://nag_raj_description/meshes/wrist_1.stl" scale="0.001 0.001 0.001"/>
-    </geometry>
-  </collision>
-</link>
-<joint name="Revolute 1" type="continuous">
-  <origin xyz="-0.001039 -0.018393 0.067132" rpy="0 0 0"/>
-  <parent link="base_link"/>
-  <child link="sh_joint_1"/>
-  <axis xyz="-0.0032 0.012661 0.999915"/>
-</joint>
-<joint name="Revolute 2" type="continuous">
-  <origin xyz="-0.092534 0.039538 0.07921" rpy="0 0 0"/>
-  <parent link="sh_joint_1"/>
-  <child link="shoulder_1"/>
-  <axis xyz="-0.922781 0.385244 -0.007831"/>
-</joint>
-<joint name="Revolute 3" type="revolute">
-  <origin xyz="0.223272 0.590898 0.077802" rpy="0 0 0"/>
-  <parent link="shoulder_1"/>
-  <child link="elbow1_1"/>
-  <axis xyz="0.922781 -0.385244 0.007831"/>
-  <limit upper="0.0" lower="-5.585054" effort="100" velocity="100"/>
-</joint>
-<joint name="Revolute 4" type="continuous">
-  <origin xyz="-0.037026 -0.223925 0.051164" rpy="0 0 0"/>
-  <parent link="elbow1_1"/>
-  <child link="elbow2_1"/>
-  <axis xyz="-0.374756 -0.892561 0.250786"/>
-</joint>
-<joint name="Revolute 5" type="continuous">
-  <origin xyz="-0.1482 -0.203372 0.05957" rpy="0 0 0"/>
-  <parent link="elbow2_1"/>
-  <child link="wrist_1"/>
-  <axis xyz="-0.924511 0.380059 -0.02887"/>
-</joint>
+  <xacro:include filename="$(find nag_raj_description)/urdf/materials.xacro" />
+  <xacro:include filename="$(find nag_raj_description)/urdf/nag_raj.trans" />
+  <xacro:include filename="$(find nag_raj_description)/urdf/nag_raj.gazebo" />
+  <link name="base_link">
+    <inertial>
+      <origin xyz="-0.0006379139080881657 -0.01809373210164651 0.030365961397063188" rpy="0 0 0" />
+      <mass value="12.627463545285623" />
+      <inertia ixx="0.031143" iyy="0.030205" izz="0.052676" ixy="-0.000405" iyz="0.000267"
+        ixz="-7e-05" />
+    </inertial>
+    <visual>
+      <origin xyz="0 0 0" rpy="0 0 0" />
+      <geometry>
+        <mesh filename="package://nag_raj_description/meshes/base_link.stl"
+          scale="0.001 0.001 0.001" />
+      </geometry>
+      <material name="silver" />
+    </visual>
+    <collision>
+      <origin xyz="0 0 0" rpy="0 0 0" />
+      <geometry>
+        <mesh filename="package://nag_raj_description/meshes/base_link.stl"
+          scale="0.001 0.001 0.001" />
+      </geometry>
+    </collision>
+  </link>
+  <link name="sh_joint_1">
+    <inertial>
+      <origin xyz="-0.0011960436685277943 0.0013481214024438706 0.07489085893279906" rpy="0 0 0" />
+      <mass value="29.69776516715868" />
+      <inertia ixx="0.099358" iyy="0.132845" izz="0.135929" ixy="0.016934" iyz="3.3e-05"
+        ixz="-0.000187" />
+    </inertial>
+    <visual>
+      <origin xyz="0.001039 0.018393 -0.067132" rpy="0 0 0" />
+      <geometry>
+        <mesh filename="package://nag_raj_description/meshes/sh_joint_1.stl"
+          scale="0.001 0.001 0.001" />
+      </geometry>
+      <material name="silver" />
+    </visual>
+    <collision>
+      <origin xyz="0.001039 0.018393 -0.067132" rpy="0 0 0" />
+      <geometry>
+        <mesh filename="package://nag_raj_description/meshes/sh_joint_1.stl"
+          scale="0.001 0.001 0.001" />
+      </geometry>
+    </collision>
+  </link>
+  <link name="shoulder_1">
+    <inertial>
+      <origin xyz="0.007821760472450007 0.2778220009300011 0.03125519386875361" rpy="0 0 0" />
+      <mass value="89.21154259038471" />
+      <inertia ixx="4.45732" iyy="1.046726" izz="5.155255" ixy="-1.710485" iyz="-0.557906"
+        ixz="-0.232136" />
+    </inertial>
+    <visual>
+      <origin xyz="0.093573 -0.021145 -0.146342" rpy="0 0 0" />
+      <geometry>
+        <mesh filename="package://nag_raj_description/meshes/shoulder_1.stl"
+          scale="0.001 0.001 0.001" />
+      </geometry>
+      <material name="silver" />
+    </visual>
+    <collision>
+      <origin xyz="0.093573 -0.021145 -0.146342" rpy="0 0 0" />
+      <geometry>
+        <mesh filename="package://nag_raj_description/meshes/shoulder_1.stl"
+          scale="0.001 0.001 0.001" />
+      </geometry>
+    </collision>
+  </link>
+  <link name="elbow1_1">
+    <inertial>
+      <origin xyz="0.012063915743866088 -0.08935136984735537 0.01819736606366848" rpy="0 0 0" />
+      <mass value="12.818945015869657" />
+      <inertia ixx="0.078237" iyy="0.022075" izz="0.079476" ixy="-0.01847" iyz="0.01453"
+        ixz="0.004333" />
+    </inertial>
+    <visual>
+      <origin xyz="-0.129699 -0.612043 -0.224144" rpy="0 0 0" />
+      <geometry>
+        <mesh filename="package://nag_raj_description/meshes/elbow1_1.stl" scale="0.001 0.001 0.001" />
+      </geometry>
+      <material name="silver" />
+    </visual>
+    <collision>
+      <origin xyz="-0.129699 -0.612043 -0.224144" rpy="0 0 0" />
+      <geometry>
+        <mesh filename="package://nag_raj_description/meshes/elbow1_1.stl" scale="0.001 0.001 0.001" />
+      </geometry>
+    </collision>
+  </link>
+  <link name="elbow2_1">
+    <inertial>
+      <origin xyz="-0.06172372576999953 -0.1471990074107003 0.039999758385676654" rpy="0 0 0" />
+      <mass value="14.074723611721877" />
+      <inertia ixx="0.09516" iyy="0.034386" izz="0.105805" ixy="-0.030922" iyz="0.020824"
+        ixz="0.008622" />
+    </inertial>
+    <visual>
+      <origin xyz="-0.092673 -0.388118 -0.275308" rpy="0 0 0" />
+      <geometry>
+        <mesh filename="package://nag_raj_description/meshes/elbow2_1.stl" scale="0.001 0.001 0.001" />
+      </geometry>
+      <material name="silver" />
+    </visual>
+    <collision>
+      <origin xyz="-0.092673 -0.388118 -0.275308" rpy="0 0 0" />
+      <geometry>
+        <mesh filename="package://nag_raj_description/meshes/elbow2_1.stl" scale="0.001 0.001 0.001" />
+      </geometry>
+    </collision>
+  </link>
+  <link name="wrist_1">
+    <inertial>
+      <origin xyz="-0.05432751125838708 0.017695228247820827 -0.0008664628207630809" rpy="0 0 0" />
+      <mass value="5.82092033198201" />
+      <inertia ixx="0.006574" iyy="0.008357" izz="0.009234" ixy="0.000912" iyz="0.000122"
+        ixz="-5e-05" />
+    </inertial>
+    <visual>
+      <origin xyz="0.055527 -0.184746 -0.334878" rpy="0 0 0" />
+      <geometry>
+        <mesh filename="package://nag_raj_description/meshes/wrist_1.stl" scale="0.001 0.001 0.001" />
+      </geometry>
+      <material name="silver" />
+    </visual>
+    <collision>
+      <origin xyz="0.055527 -0.184746 -0.334878" rpy="0 0 0" />
+      <geometry>
+        <mesh filename="package://nag_raj_description/meshes/wrist_1.stl" scale="0.001 0.001 0.001" />
+      </geometry>
+    </collision>
+  </link>
+  <joint name="Revolute 1" type="continuous">
+    <origin xyz="-0.001039 -0.018393 0.067132" rpy="0 0 0" />
+    <parent link="base_link" />
+    <child link="sh_joint_1" />
+    <axis xyz="-0.0032 0.012661 0.999915" />
+  </joint>
+  <joint name="Revolute 2" type="continuous">
+    <origin xyz="-0.092534 0.039538 0.07921" rpy="0 0 0" />
+    <parent link="sh_joint_1" />
+    <child link="shoulder_1" />
+    <axis xyz="-0.922781 0.385244 -0.007831" />
+  </joint>
+  <joint name="Revolute 3" type="revolute">
+    <origin xyz="0.223272 0.590898 0.077802" rpy="0 0 0" />
+    <parent link="shoulder_1" />
+    <child link="elbow1_1" />
+    <axis xyz="0.922781 -0.385244 0.007831" />
+    <limit upper="0.0" lower="-5.585054" effort="100" velocity="100" />
+  </joint>
+  <joint name="Revolute 4" type="continuous">
+    <origin xyz="-0.037026 -0.223925 0.051164" rpy="0 0 0" />
+    <parent link="elbow1_1" />
+    <child link="elbow2_1" />
+    <axis xyz="-0.374756 -0.892561 0.250786" />
+  </joint>
+  <joint name="Revolute 5" type="continuous">
+    <origin xyz="-0.1482 -0.203372 0.05957" rpy="0 0 0" />
+    <parent link="elbow2_1" />
+    <child link="wrist_1" />
+    <axis xyz="-0.924511 0.380059 -0.02887" />
+  </joint>
+  <link name="kinect">
+    <collision>
+      <origin xyz="0 0 0" rpy="1.57 0 0" />
+      <geometry>
+        <mesh filename="package://nag_raj_description/meshes/kinect.stl" scale="0.005 0.005 0.005" />
+      </geometry>
+    </collision>
+    <visual>
+      <origin xyz="0 0 0" rpy="1.57 1.57 0" />
+      <geometry>
+        <mesh filename="package://nag_raj_description/meshes/kinect.stl" scale="0.005 0.005 0.005" />
+      </geometry>
+    </visual>
+    <inertial>
+      <mass value="1e-5" />
+      <origin xyz="0 0 0" rpy="0 0 0" />
+      <inertia ixx="1e-6" ixy="0" ixz="0" iyy="1e-6" iyz="0" izz="1e-6" />
+    </inertial>
+  </link>
+  <joint name="kinect_joint" type="fixed">
+    <origin xyz="1 0 3" rpy="0 1.57 0" />
+    <parent link="base_link" />
+    <child link="kinect" />
+  </joint>
 </robot>

Commit message: kinect point-cloud data received successfully

File: nag_raj_description/urdf/nag_raj.xacro (robot description, xacro)
@@ -175,5 +175,5 @@
     </collision>
     <visual>
-      <origin xyz="0 0 0" rpy="1.57 1.57 0" />
+      <origin xyz="0 0 0" rpy="1.57 -1.57 0" />
       <geometry>
         <mesh filename="package://nag_raj_description/meshes/kinect.stl" scale="0.005 0.005 0.005" />

Commit message: Modify Kinect position

File: nag_raj_description/urdf/nag_raj.xacro (robot description, xacro)
@@ -187,5 +187,5 @@
   </link>
   <joint name="kinect_joint" type="fixed">
-    <origin xyz="1 0 3" rpy="0 1.57 0" />
+    <origin xyz="-0.8 0 1.5" rpy="0 1.57 0" />
     <parent link="base_link" />
     <child link="kinect" />
