Commit message: new urdf added with test service scripts

File: ajgar/urdf/ajgar_URDF.xacro (robot description, xacro)
@@ -7,7 +7,7 @@
 <link name="base_link">
   <inertial>
-    <origin xyz="0.006181560825936428 0.03299945212996641 0.024980891310047913" rpy="0 0 0"/>
-    <mass value="8.92124295451605"/>
-    <inertia ixx="0.018904" iyy="0.023843" izz="0.038855" ixy="-0.0" iyz="-1e-06" ixz="0.000101"/>
+    <origin xyz="-0.00865082588772432 1.8113911902102217e-07 0.032368373908884494" rpy="0 0 0"/>
+    <mass value="9.059758934586307"/>
+    <inertia ixx="0.021583" iyy="0.026795" izz="0.042202" ixy="-0.0" iyz="-0.0" ixz="0.000269"/>
   </inertial>
   <visual>
@@ -27,10 +27,10 @@
 <link name="base_top">
   <inertial>
-    <origin xyz="3.7368745492756403e-06 0.0001746213937584215 0.03246703696650755" rpy="0 0 0"/>
-    <mass value="1.2219948495058053"/>
-    <inertia ixx="0.001733" iyy="0.001362" izz="0.001507" ixy="1e-06" iyz="2.5e-05" ixz="1e-06"/>
+    <origin xyz="1.279003402099646e-05 -0.0022856514871783416 0.03289309768621855" rpy="0 0 0"/>
+    <mass value="1.4850383611977547"/>
+    <inertia ixx="0.002124" iyy="0.00176" izz="0.001747" ixy="-0.0" iyz="0.000118" ixz="0.0"/>
   </inertial>
   <visual>
-    <origin xyz="-0.0 -0.033 -0.049132" rpy="0 0 0"/>
+    <origin xyz="0.015013 -0.0 -0.06" rpy="0 0 0"/>
     <geometry>
       <mesh filename="package://ajgar/meshes/base_top.stl" scale="0.001 0.001 0.001"/>
@@ -39,5 +39,5 @@
   </visual>
   <collision>
-    <origin xyz="-0.0 -0.033 -0.049132" rpy="0 0 0"/>
+    <origin xyz="0.015013 -0.0 -0.06" rpy="0 0 0"/>
     <geometry>
       <mesh filename="package://ajgar/meshes/base_top.stl" scale="0.001 0.001 0.001"/>
@@ -47,10 +47,10 @@
 <link name="shoulder">
   <inertial>
-    <origin xyz="-5.812758879132124e-06 0.0302940521651806 0.10674081963818186" rpy="0 0 0"/>
-    <mass value="2.9743567366826063"/>
-    <inertia ixx="0.027269" iyy="0.027148" izz="0.002649" ixy="1e-06" iyz="0.00023" ixz="3e-06"/>
+    <origin xyz="1.2461762721963782e-06 0.025783530669485587 0.11928257744286477" rpy="0 0 0"/>
+    <mass value="2.8383656665985857"/>
+    <inertia ixx="0.03026" iyy="0.030184" izz="0.00245" ixy="-0.0" iyz="0.000773" ixz="0.0"/>
   </inertial>
   <visual>
-    <origin xyz="-0.0 -0.008 -0.102632" rpy="0 0 0"/>
+    <origin xyz="0.015013 0.025 -0.119368" rpy="0 0 0"/>
     <geometry>
       <mesh filename="package://ajgar/meshes/shoulder.stl" scale="0.001 0.001 0.001"/>
@@ -59,5 +59,5 @@
   </visual>
   <collision>
-    <origin xyz="-0.0 -0.008 -0.102632" rpy="0 0 0"/>
+    <origin xyz="0.015013 0.025 -0.119368" rpy="0 0 0"/>
     <geometry>
       <mesh filename="package://ajgar/meshes/shoulder.stl" scale="0.001 0.001 0.001"/>
@@ -65,12 +65,52 @@
   </collision>
 </link>
+<link name="elbow">
+  <inertial>
+    <origin xyz="-0.0003292153850686253 0.026723336517713626 0.10654902767889785" rpy="0 0 0"/>
+    <mass value="2.4072821039747727"/>
+    <inertia ixx="0.026455" iyy="0.026758" izz="0.001672" ixy="-4e-06" iyz="0.000315" ixz="0.000123"/>
+  </inertial>
+  <visual>
+    <origin xyz="0.015013 0.025 -0.377365" rpy="0 0 0"/>
+    <geometry>
+      <mesh filename="package://ajgar/meshes/elbow.stl" scale="0.001 0.001 0.001"/>
+    </geometry>
+    <material name="silver"/>
+  </visual>
+  <collision>
+    <origin xyz="0.015013 0.025 -0.377365" rpy="0 0 0"/>
+    <geometry>
+      <mesh filename="package://ajgar/meshes/elbow.stl" scale="0.001 0.001 0.001"/>
+    </geometry>
+  </collision>
+</link>
+<link name="wrist">
+  <inertial>
+    <origin xyz="0.00920373509392226 -0.01118771679377522 0.025837849583827288" rpy="0 0 0"/>
+    <mass value="0.34678950211541076"/>
+    <inertia ixx="0.000595" iyy="0.000274" izz="0.000554" ixy="9.5e-05" iyz="7.4e-05" ixz="-6e-05"/>
+  </inertial>
+  <visual>
+    <origin xyz="0.015013 -0.0 -0.644865" rpy="0 0 0"/>
+    <geometry>
+      <mesh filename="package://ajgar/meshes/wrist.stl" scale="0.001 0.001 0.001"/>
+    </geometry>
+    <material name="silver"/>
+  </visual>
+  <collision>
+    <origin xyz="0.015013 -0.0 -0.644865" rpy="0 0 0"/>
+    <geometry>
+      <mesh filename="package://ajgar/meshes/wrist.stl" scale="0.001 0.001 0.001"/>
+    </geometry>
+  </collision>
+</link>
 <link name="suction">
   <inertial>
-    <origin xyz="0.0013549004342596088 0.036865135906333266 0.0010284048884452446" rpy="0 0 0"/>
-    <mass value="1.0937894888063466"/>
-    <inertia ixx="0.000604" iyy="0.000571" izz="0.000737" ixy="-6e-06" iyz="-1e-06" ixz="2.3e-05"/>
+    <origin xyz="-8.479527444330004e-05 0.03652030172582285 8.898889773256702e-05" rpy="0 0 0"/>
+    <mass value="0.6053245769138885"/>
+    <inertia ixx="0.000476" iyy="0.000398" izz="0.000554" ixy="0.0" iyz="-0.0" ixz="1.7e-05"/>
   </inertial>
   <visual>
-    <origin xyz="-0.0 -0.001 -0.645153" rpy="0 0 0"/>
+    <origin xyz="0.015013 0.037 -0.689865" rpy="0 0 0"/>
     <geometry>
       <mesh filename="package://ajgar/meshes/suction.stl" scale="0.001 0.001 0.001"/>
@@ -79,5 +119,5 @@
   </visual>
   <collision>
-    <origin xyz="-0.0 -0.001 -0.645153" rpy="0 0 0"/>
+    <origin xyz="0.015013 0.037 -0.689865" rpy="0 0 0"/>
     <geometry>
       <mesh filename="package://ajgar/meshes/suction.stl" scale="0.001 0.001 0.001"/>
@@ -85,72 +125,12 @@
   </collision>
 </link>
-<link name="camera_link">
+<link name="end">
   <inertial>
-    <origin xyz="0.028614791844949194 4.630497056100358e-05 -0.041124324616634844" rpy="0 0 0"/>
-    <mass value="5.170558909547441"/>
-    <inertia ixx="0.024426" iyy="0.003279" izz="0.024604" ixy="-1e-06" iyz="8e-06" ixz="1.9e-05"/>
+    <origin xyz="-9.118561992635388e-08 3.576502294322381e-10 -0.00900061967229826" rpy="0 0 0"/>
+    <mass value="0.07630173554088619"/>
+    <inertia ixx="7e-06" iyy="5e-06" izz="8e-06" ixy="0.0" iyz="-0.0" ixz="0.0"/>
   </inertial>
   <visual>
-    <origin xyz="-0.432718 -0.043482 -0.770132" rpy="0 0 0"/>
-    <geometry>
-      <mesh filename="package://ajgar/meshes/KINECT_XBOX.stl" scale="0.001 0.001 0.001"/>
-    </geometry>
-    <material name="silver"/>
-  </visual>
-  <collision>
-    <origin xyz="-0.432718 -0.043482 -0.770132" rpy="0 0 0"/>
-    <geometry>
-      <mesh filename="package://ajgar/meshes/KINECT_XBOX.stl" scale="0.001 0.001 0.001"/>
-    </geometry>
-  </collision>
-</link>
-<link name="wrist">
-  <inertial>
-    <origin xyz="0.0008459460576890564 0.00015757637059889834 0.0167203860599896" rpy="0 0 0"/>
-    <mass value="1.2638223022450714"/>
-    <inertia ixx="0.001154" iyy="0.001222" izz="0.000623" ixy="-7e-06" iyz="-2e-06" ixz="1.3e-05"/>
-  </inertial>
-  <visual>
-    <origin xyz="-0.0 -0.038 -0.545632" rpy="0 0 0"/>
-    <geometry>
-      <mesh filename="package://ajgar/meshes/wrist.stl" scale="0.001 0.001 0.001"/>
-    </geometry>
-    <material name="silver"/>
-  </visual>
-  <collision>
-    <origin xyz="-0.0 -0.038 -0.545632" rpy="0 0 0"/>
-    <geometry>
-      <mesh filename="package://ajgar/meshes/wrist.stl" scale="0.001 0.001 0.001"/>
-    </geometry>
-  </collision>
-</link>
-<link name="extrusion3">
-  <inertial>
-    <origin xyz="0.30550252641395526 -0.019853978999297 0.5577011626661099" rpy="0 0 0"/>
-    <mass value="5.889005305436553"/>
-    <inertia ixx="1.15866" iyy="0.40406" izz="0.755642" ixy="0.00111" iyz="-0.003566" ixz="0.000389"/>
-  </inertial>
-  <visual>
-    <origin xyz="-0.136552 -0.066 0.029236" rpy="0 0 0"/>
-    <geometry>
-      <mesh filename="package://ajgar/meshes/extrusion3.stl" scale="0.001 0.001 0.001"/>
-    </geometry>
-    <material name="silver"/>
-  </visual>
-  <collision>
-    <origin xyz="-0.136552 -0.066 0.029236" rpy="0 0 0"/>
-    <geometry>
-      <mesh filename="package://ajgar/meshes/extrusion3.stl" scale="0.001 0.001 0.001"/>
-    </geometry>
-  </collision>
-</link>
-<link name="end">
-  <inertial>
-    <origin xyz="1.599846658410097e-05 -0.02828005788406872 0.034985952571814805" rpy="0 0 0"/>
-    <mass value="0.6717186078596652"/>
-    <inertia ixx="0.001219" iyy="0.000367" izz="0.00104" ixy="2e-06" iyz="0.00019" ixz="-2e-06"/>
-  </inertial>
-  <visual>
-    <origin xyz="-0.0 -0.038 -0.600132" rpy="0 0 0"/>
+    <origin xyz="0.015013 -0.0 -0.714365" rpy="0 0 0"/>
     <geometry>
       <mesh filename="package://ajgar/meshes/end.stl" scale="0.001 0.001 0.001"/>
@@ -159,5 +139,5 @@
   </visual>
   <collision>
-    <origin xyz="-0.0 -0.038 -0.600132" rpy="0 0 0"/>
+    <origin xyz="0.015013 -0.0 -0.714365" rpy="0 0 0"/>
     <geometry>
       <mesh filename="package://ajgar/meshes/end.stl" scale="0.001 0.001 0.001"/>
@@ -165,78 +145,50 @@
   </collision>
 </link>
-<link name="elbow">
-  <inertial>
-    <origin xyz="2.557388937857749e-06 0.027722993563970767 0.0338440776447978" rpy="0 0 0"/>
-    <mass value="1.503376993994313"/>
-    <inertia ixx="0.004533" iyy="0.004824" izz="0.001216" ixy="-0.0" iyz="2.3e-05" ixz="-0.0"/>
-  </inertial>
-  <visual>
-    <origin xyz="-0.0 -0.013 -0.340632" rpy="0 0 0"/>
-    <geometry>
-      <mesh filename="package://ajgar/meshes/elbow.stl" scale="0.001 0.001 0.001"/>
-    </geometry>
-    <material name="silver"/>
-  </visual>
-  <collision>
-    <origin xyz="-0.0 -0.013 -0.340632" rpy="0 0 0"/>
-    <geometry>
-      <mesh filename="package://ajgar/meshes/elbow.stl" scale="0.001 0.001 0.001"/>
-    </geometry>
-  </collision>
-</link>
-<joint name="world_joint" type="fixed">
-    <parent link="world" />
-    <child link="base_link" />
-    <origin rpy="0 0 3.142" xyz="0.0 0.0 0.0" />
+<joint name="world_joint  " type="fixed">
+  <parent link="world" />
+  <child link="base_link" />
+  <origin rpy="0 0 3.142" xyz="0.0 0.0 0.0" />
 </joint>
 <joint name="base_joint" type="revolute">
-  <origin xyz="0.0 0.033 0.049132" rpy="0 0 0"/>
+  <origin xyz="-0.015013 0.0 0.06" rpy="0 0 0"/>
   <parent link="base_link"/>
   <child link="base_top"/>
-  <axis xyz="-0.0 0.0 1.0"/>
-  <limit upper="2.443461" lower="-2.443461" effort="100" velocity="100"/>
+  <axis xyz="0.0 0.0 1.0"/>
+  <limit upper="2.879793" lower="-2.879793" effort="100" velocity="100" />
 </joint>
 <joint name="shoulder_joint" type="revolute">
-  <origin xyz="0.0 -0.025 0.0535" rpy="0 0 0"/>
+  <origin xyz="0.0 -0.025 0.059368" rpy="0 0 0"/>
   <parent link="base_top"/>
   <child link="shoulder"/>
-  <axis xyz="-0.0 1.0 -0.0"/>
-  <limit upper="1.570796" lower="-1.570796" effort="100" velocity="100"/>
+  <axis xyz="0.0 -1.0 0.0"/>
+  <limit upper="1.57" lower="-1.57" effort="100" velocity="100" />
 </joint>
-<joint name="wrist_joint" type="fixed">
-  <origin xyz="0.0 0.025 0.205" rpy="0 0 0"/>
+<joint name="arm_joint" type="revolute">
+  <origin xyz="0.0 0.0 0.257997" rpy="0 0 0"/>
+  <parent link="shoulder"/>
+  <child link="elbow"/>
+  <axis xyz="0.0 -1.0 -0.0"/>
+  <limit upper="1.57" lower="-1.57" effort="100" velocity="100" />
+</joint>
+<joint name="forearm_joint" type="revolute">
+  <origin xyz="0.0 0.025 0.2675" rpy="0 0 0"/>
   <parent link="elbow"/>
   <child link="wrist"/>
+  <axis xyz="-0.0 0.0 1.0"/>
+  <limit upper="2.879793" lower="-2.879793" effort="100" velocity="100" />
 </joint>
-<joint name="forearm_joint" type="revolute">
-  <origin xyz="0.0 0.0 0.0545" rpy="0 0 0"/>
+<joint name="end_joint" type="revolute">
+  <origin xyz="0.0 -0.037 0.045" rpy="0 0 0"/>
   <parent link="wrist"/>
-  <child link="end"/>
-  <axis xyz="-0.0 -0.0 1.0"/>
-  <limit upper="2.443461" lower="-2.443461" effort="100" velocity="100"/>
-</joint>
-<joint name="elbow_joint" type="revolute">
-  <origin xyz="0.0 0.005 0.238" rpy="0 0 0"/>
-  <parent link="shoulder"/>
-  <child link="elbow"/>
+  <child link="suction"/>
   <axis xyz="-0.0 1.0 -0.0"/>
-  <limit upper="2.443461" lower="-2.443461" effort="100" velocity="100"/>
+  <limit upper="2.879793" lower="-2.879793" effort="100" velocity="100" />
 </joint>
 <joint name="suction_joint" type="revolute">
-  <origin xyz="0.0 -0.037 0.045021" rpy="0 0 0"/>
-  <parent link="end"/>
-  <child link="suction"/>
-  <axis xyz="0.0 -1.0 0.0"/>
-  <limit upper="2.443461" lower="-0.698132" effort="100" velocity="100"/>
-</joint>
-<joint name="kinect_joint" type="fixed">
-  <origin xyz="0.296166 -0.022518 0.799368" rpy="0 -4.6 0"/>
-  <parent link="extrusion3"/>
-  <child link="camera_link"/>
-</joint>
-<joint name="extrusion_joint" type="fixed">
-  <origin xyz="0.136552 0.066 -0.029236" rpy="0 0 0"/>
-  <parent link="base_link"/>
-  <child link="extrusion3"/>
+  <origin xyz="0.0 0.037 0.0245" rpy="0 0 0"/>
+  <parent link="suction"/>
+  <child link="end"/>
+  <axis xyz="-0.0 -0.0 -1.0"/>
+  <limit upper="2.879793" lower="-2.879793" effort="100" velocity="100" />
 </joint>
 </robot>

File: ajgar/urdf/materials.xacro (robot description, xacro)
@@ -1,4 +1,4 @@
 <?xml version="1.0" ?>
-<robot name="test" xmlns:xacro="http://www.ros.org/wiki/xacro" >
+<robot name="ajgar" xmlns:xacro="http://www.ros.org/wiki/xacro" >
 <material name="silver">
   <color rgba="0.700 0.700 0.700 1.000"/>

File: ajgar_moveit_config/config/gazebo_ajgar.urdf (robot description, URDF)
Before this commit: robot ajgar, 10 links, 9 joints
Links:
- removed link camera_link
- removed link extrusion3
- removed link world
- link base_link: mass 8.92124295451605 -> 9.059758934586307
- link base_top: mass 1.2219948495058053 -> 1.4850383611977547
- link elbow: mass 1.503376993994313 -> 2.4072821039747727
- link end: mass 0.6717186078596652 -> 0.07630173554088619
- link shoulder: mass 2.9743567366826063 -> 2.8383656665985857
- link suction: mass 1.0937894888063466 -> 0.6053245769138885
- link wrist: mass 1.2638223022450714 -> 0.34678950211541076
Joints:
- removed joint elbow_joint
- removed joint extrusion_joint
- removed joint kinect_joint
- removed joint world_joint
- removed joint wrist_joint
- added joint arm_joint: type continuous, parent shoulder, child elbow, origin xyz=0.0 0.0 0.257997 rpy=0 0 0, axis 0.0 -1.0 -0.0
- added joint end_joint: type continuous, parent wrist, child suction, origin xyz=0.0 -0.037 0.045 rpy=0 0 0, axis -0.0 1.0 -0.0
- joint base_joint: axis -0.0 0.0 1.0 -> 0.0 0.0 1.0; origin xyz=0.0 0.033 0.049132 rpy=0 0 0 -> xyz=-0.015013 0.0 0.06 rpy=0 0 0
- joint forearm_joint: axis -0.0 -0.0 1.0 -> -0.0 0.0 1.0; child end -> wrist; origin xyz=0.0 0.0 0.0545 rpy=0 0 0 -> xyz=0.0 0.025 0.2675 rpy=0 0 0; parent wrist -> elbow
- joint shoulder_joint: axis -0.0 1.0 -0.0 -> 0.0 -1.0 0.0; limit lower=-1.570796 upper=1.570796 effort=100 velocity=100 -> (none); origin xyz=0.0 -0.025 0.0535 rpy=0 0 0 -> xyz=0.0 -0.025 0.059368 rpy=0 0 0; type revolute -> continuous
- joint suction_joint: axis 0.0 -1.0 0.0 -> -0.0 -0.0 -1.0; child suction -> end; limit lower=-0.698132 upper=2.443461 effort=100 velocity=100 -> (none); origin xyz=0.0 -0.037 0.045021 rpy=0 0 0 -> xyz=0.0 0.037 0.0245 rpy=0 0 0; parent end -> suction; type revolute -> continuous
