Commit message: fixed the kinect urdf issue

File: ajgar_moveit_config/config/gazebo_ajgar.urdf (robot description, URDF)
Before this commit: robot ajgar, 10 links, 9 joints
Links:
- removed link KINECT_XBOX
- added link camera_link, mass 5.170558909547441; collision mesh filename=package://ajgar/meshes/KINECT_XBOX.stl scale=0.001 0.001 0.001; visual mesh filename=package://ajgar/meshes/KINECT_XBOX.stl scale=0.001 0.001 0.001
Joints:
- joint kinect_joint: child KINECT_XBOX -> camera_link

Commit message: organized the repository and removed unnecessary files

File: ajgar_moveit_config/config/gazebo_ajgar.urdf (robot description, URDF)
Before this commit: robot ajgar, 7 links, 6 joints
Links:
- removed link arm_1
- removed link end_1
- removed link forearm_1
- removed link shoulder_1
- removed link suction_1
- removed link wrist_1
- added link base_top, mass 0.446819319233817; collision mesh filename=package://ajgar/meshes/base_top.stl scale=0.001 0.001 0.001; visual mesh filename=package://ajgar/meshes/base_top.stl scale=0.001 0.001 0.001
- added link elbow, mass 2.365159547256585; collision mesh filename=package://ajgar/meshes/elbow.stl scale=0.001 0.001 0.001; visual mesh filename=package://ajgar/meshes/elbow.stl scale=0.001 0.001 0.001
- added link end, mass 0.07642686015416068; collision mesh filename=package://ajgar/meshes/end.stl scale=0.001 0.001 0.001; visual mesh filename=package://ajgar/meshes/end.stl scale=0.001 0.001 0.001
- added link shoulder, mass 4.919783093355411; collision mesh filename=package://ajgar/meshes/shoulder.stl scale=0.001 0.001 0.001; visual mesh filename=package://ajgar/meshes/shoulder.stl scale=0.001 0.001 0.001
- added link suction, mass 0.605324576914463; collision mesh filename=package://ajgar/meshes/suction.stl scale=0.001 0.001 0.001; visual mesh filename=package://ajgar/meshes/suction.stl scale=0.001 0.001 0.001
- added link world
- added link wrist, mass 0.338076325355839; collision mesh filename=package://ajgar/meshes/wrist.stl scale=0.001 0.001 0.001; visual mesh filename=package://ajgar/meshes/wrist.stl scale=0.001 0.001 0.001
- link base_link: mass 29.485735477923164 -> 5.004539313789304
Joints:
- removed joint arm_joint
- removed joint base_joint
- removed joint forearm_joint
- removed joint suction_joint
- removed joint wrist_joint
- added joint base: type continuous, parent base_link, child base_top, origin xyz=0.0 0.0 0.049 rpy=0 0 0, axis -0.0 0.0 1.0
- added joint elbow_joint: type continuous, parent shoulder, child elbow, origin xyz=0.000405 0.058 0.278851 rpy=0 0 0, axis 0.0 -1.0 0.0
- added joint end_joint: type continuous, parent suction, child end, origin xyz=0.0 0.037 0.0245 rpy=0 0 0, axis -0.0 -0.0 -1.0
- added joint lower_wrist_joint: type continuous, parent elbow, child wrist, origin xyz=0.0 -0.028 0.2 rpy=0 0 0, axis 0.0 0.0 1.0
- added joint upper_wrist_joint: type continuous, parent wrist, child suction, origin xyz=0.0 -0.037 0.045 rpy=0 0 0, axis -0.0 1.0 -0.0
- added joint world_joint: type fixed, parent world, child base_link, origin xyz=0.0 0.0 0.0 rpy=0 0 3.142
- joint shoulder_joint: axis -0.0 -1.0 0.0 -> -0.0 1.0 -0.0; child arm_1 -> shoulder; origin xyz=0.0 -0.0946 0.0814 rpy=0 0 0 -> xyz=-0.005001 -0.03 0.125627 rpy=0 0 0; parent shoulder_1 -> base_top
