Commit message: modifed arm position wrt trolley

File: ajgar_core/scripts/ajgar.xacro (robot description, xacro)
@@ -1,4 +1,4 @@
 <?xml version="1.0" ?>
-<robot name="ajgar_description" xmlns:xacro="http://www.ros.org/wiki/xacro">
+<robot name="ajgar" xmlns:xacro="http://www.ros.org/wiki/xacro">
 <xacro:include filename="$(find ajgar_description)/urdf/materials.xacro" />
 <xacro:include filename="$(find ajgar_description)/urdf/ajgar.trans" />
@@ -212,5 +212,5 @@
 </joint>
 <joint name="kinect_joint" type="fixed">
-  <origin xyz="0.612 -0.15 1.5" rpy="0 1.57 0" />
+  <origin xyz="0.60 -0.15 1.3" rpy="0 1.57 0" />
   <parent link="base_link" />
   <child link="camera_depth_frame" />

File: ajgar_description/urdf/ajgar.xacro (robot description, xacro)
@@ -1,4 +1,4 @@
 <?xml version="1.0" ?>
-<robot name="ajgar_description" xmlns:xacro="http://www.ros.org/wiki/xacro">
+<robot name="ajgar" xmlns:xacro="http://www.ros.org/wiki/xacro">
 <xacro:include filename="$(find ajgar_description)/urdf/materials.xacro" />
 <xacro:include filename="$(find ajgar_description)/urdf/ajgar.trans" />
@@ -212,5 +212,5 @@
 </joint>
 <joint name="kinect_joint" type="fixed">
-  <origin xyz="0.612 -0.15 1.5" rpy="0 1.57 0" />
+  <origin xyz="0.612 0.0 1.5" rpy="0 1.57 0" />
   <parent link="base_link" />
   <child link="camera_depth_frame" />

Commit message: new world generated

File: ajgar_core/scripts/ajgar.xacro (robot description, xacro)
@@ -125,5 +125,5 @@
   </collision>
 </link>
-<link name="end">
+<!-- <link name="end">
   <inertial>
     <origin xyz="-8.702208040972659e-08 -2.1072130740783367e-09 0.005896611642581373" rpy="0 0 0"/>
@@ -144,6 +144,6 @@
     </geometry>
   </collision>
-</link>
-<link name="camera_depth_frame">
+</link> -->
+<link name="camera_link">
     <collision>
       <origin xyz="0 0 0" rpy="1.57 0 0" />
@@ -214,5 +214,5 @@
   <origin xyz="0.60 -0.15 1.3" rpy="0 1.57 0" />
   <parent link="base_link" />
-  <child link="camera_depth_frame" />
+  <child link="camera_link" />
 </joint>
 </robot>

File: ajgar_core/scripts/arm.urdf (robot description, URDF)
Before this commit: robot ajgar, 9 links, 8 joints
Links:
- removed link camera_depth_frame
- added link camera_link, mass 1e-5; collision mesh filename=package://ur5_description/meshes/kinect.stl scale=0.005 0.005 0.005; visual mesh filename=package://ur5_description/meshes/kinect.stl scale=0.005 0.005 0.005
Joints:
- joint kinect_joint: child camera_depth_frame -> camera_link; origin xyz=0.612 -0.15 1.5 rpy=0 1.57 0 -> xyz=0.40 0.0 1.0 rpy=0 1.57 0

File: ajgar_description/urdf/ajgar.xacro (robot description, xacro)
@@ -145,5 +145,5 @@
   </collision>
 </link>
-<link name="camera_depth_frame">
+<link name="camera_link">
   <collision>
     <origin xyz="0 0 0" rpy="1.57 0 0" />
@@ -212,7 +212,7 @@
 </joint>
 <joint name="kinect_joint" type="fixed">
-  <origin xyz="0.612 0.0 1.5" rpy="0 1.57 0" />
+  <origin xyz="0.40 0.0 1.0" rpy="0 1.57 0" />
   <parent link="base_link" />
-  <child link="camera_depth_frame" />
+  <child link="camera_link" />
 </joint>
 </robot>
