Commit message: added track_ik solver pkg

File: ajgar_description/urdf/ajgar.xacro (robot description, xacro)
@@ -150,39 +150,45 @@
     <origin rpy="0 0 3.142" xyz="0.0 0.0 0.0" />
 </joint>
-<joint name="base" type="continuous">
+<joint name="base" type="revolute">
   <origin xyz="0.0 0.0 0.049" rpy="0 0 0"/>
   <parent link="base_link"/>
   <child link="base_top"/>
   <axis xyz="-0.0 0.0 1.0"/>
+  <limit upper="2.879793" lower="-2.879793" effort="100" velocity="100" />
 </joint>
-<joint name="shoulder_joint" type="continuous">
+<joint name="shoulder_joint" type="revolute">
   <origin xyz="-0.005001 -0.03 0.125627" rpy="0 0 0"/>
   <parent link="base_top"/>
   <child link="shoulder"/>
   <axis xyz="-0.0 1.0 -0.0"/>
+  <limit upper="2.879793" lower="-2.879793" effort="100" velocity="100" />
 </joint>
-<joint name="elbow_joint" type="continuous">
+<joint name="elbow_joint" type="revolute">
   <origin xyz="0.000405 0.058 0.278851" rpy="0 0 0"/>
   <parent link="shoulder"/>
   <child link="elbow"/>
   <axis xyz="0.0 -1.0 0.0"/>
+  <limit upper="2.879793" lower="-2.879793" effort="100" velocity="100" />
 </joint>
-<joint name="lower_wrist_joint" type="continuous">
+<joint name="lower_wrist_joint" type="revolute">
   <origin xyz="0.0 -0.028 0.2" rpy="0 0 0"/>
   <parent link="elbow"/>
   <child link="wrist"/>
   <axis xyz="0.0 0.0 1.0"/>
+    <limit upper="2.879793" lower="-2.879793" effort="100" velocity="100" />
 </joint>
-<joint name="upper_wrist_joint" type="continuous">
+<joint name="upper_wrist_joint" type="revolute">
   <origin xyz="0.0 -0.037 0.045" rpy="0 0 0"/>
   <parent link="wrist"/>
   <child link="suction"/>
   <axis xyz="-0.0 1.0 -0.0"/>
+    <limit upper="2.879793" lower="-2.879793" effort="100" velocity="100" />
 </joint>
-<joint name="end_joint" type="continuous">
+<joint name="end_joint" type="revolute">
   <origin xyz="0.0 0.037 0.0245" rpy="0 0 0"/>
   <parent link="suction"/>
   <child link="end"/>
   <axis xyz="-0.0 -0.0 -1.0"/>
+    <limit upper="2.879793" lower="-2.879793" effort="100" velocity="100" />
 </joint>
 </robot>

Commit message: arm motion automated using trac_ik

File: ajgar_description/urdf/ajgar.xacro (robot description, xacro)
@@ -155,5 +155,5 @@
   <child link="base_top"/>
   <axis xyz="-0.0 0.0 1.0"/>
-  <limit upper="2.879793" lower="-2.879793" effort="100" velocity="100" />
+  <limit upper="3.14159" lower="-3.14159" effort="100" velocity="100" />
 </joint>
 <joint name="shoulder_joint" type="revolute">
@@ -162,5 +162,5 @@
   <child link="shoulder"/>
   <axis xyz="-0.0 1.0 -0.0"/>
-  <limit upper="2.879793" lower="-2.879793" effort="100" velocity="100" />
+  <limit upper="2.16421" lower="-2.33874" effort="100" velocity="100" />
 </joint>
 <joint name="elbow_joint" type="revolute">
@@ -169,5 +169,5 @@
   <child link="elbow"/>
   <axis xyz="0.0 -1.0 0.0"/>
-  <limit upper="2.879793" lower="-2.879793" effort="100" velocity="100" />
+  <limit upper="2.79253" lower="-2.79253" effort="100" velocity="100" />
 </joint>
 <joint name="lower_wrist_joint" type="revolute">
@@ -176,5 +176,5 @@
   <child link="wrist"/>
   <axis xyz="0.0 0.0 1.0"/>
-    <limit upper="2.879793" lower="-2.879793" effort="100" velocity="100" />
+    <limit upper="3.14159" lower="-3.14159" effort="100" velocity="100" />
 </joint>
 <joint name="upper_wrist_joint" type="revolute">
@@ -183,5 +183,5 @@
   <child link="suction"/>
   <axis xyz="-0.0 1.0 -0.0"/>
-    <limit upper="2.879793" lower="-2.879793" effort="100" velocity="100" />
+    <limit upper="0.837758" lower="-2.58309" effort="100" velocity="100" />
 </joint>
 <joint name="end_joint" type="revolute">
@@ -190,5 +190,5 @@
   <child link="end"/>
   <axis xyz="-0.0 -0.0 -1.0"/>
-    <limit upper="2.879793" lower="-2.879793" effort="100" velocity="100" />
+    <limit upper="3.14159" lower="-3.14159" effort="100" velocity="100" />
 </joint>
 </robot>

File: trac_ik/trac_ik_python/scripts/arm.urdf (robot description, URDF)
Before this commit: robot ajgar_description, 8 links, 7 joints
Joints:
- joint base: limit lower=-2.879793 upper=2.879793 effort=100 velocity=100 -> lower=-3.14159 upper=3.14159 effort=100 velocity=100
- joint elbow_joint: limit lower=-2.879793 upper=2.879793 effort=100 velocity=100 -> lower=-2.79253 upper=2.79253 effort=100 velocity=100
- joint end_joint: limit lower=-2.879793 upper=2.879793 effort=100 velocity=100 -> lower=-3.14159 upper=3.14159 effort=100 velocity=100
- joint lower_wrist_joint: limit lower=-2.879793 upper=2.879793 effort=100 velocity=100 -> lower=-3.14159 upper=3.14159 effort=100 velocity=100
- joint shoulder_joint: limit lower=-2.879793 upper=2.879793 effort=100 velocity=100 -> lower=-2.33874 upper=2.16421 effort=100 velocity=100
- joint upper_wrist_joint: limit lower=-2.879793 upper=2.879793 effort=100 velocity=100 -> lower=-2.58309 upper=0.837758 effort=100 velocity=100

Commit message: corrected tf tree

File: ajgar_description/urdf/ajgar.xacro (robot description, xacro)
@@ -145,5 +145,5 @@
   </collision>
 </link>
-<link name="camera_depth_frame">
+<link name="camera_link">
     <collision>
       <origin xyz="0 0 0" rpy="1.57 0 0" />
@@ -214,5 +214,5 @@
   <origin xyz="0.612 -0.15 1.5" rpy="0 1.57 0" />
   <parent link="base_link" />
-  <child link="camera_depth_frame" />
+  <child link="camera_link" />
 </joint>
 </robot>

File: ur5_description/urdf/ur5.xacro (robot description, xacro)
@@ -146,5 +146,5 @@
     </collision>
   </link>
-  <link name="camera_depth_frame">
+  <link name="camera_link">
     <collision>
       <origin xyz="0 0 0" rpy="1.57 0 0" />
@@ -215,5 +215,5 @@
     <origin xyz="0.612 -0.15 1.5" rpy="0 1.57 0" />
     <parent link="base_link" />
-    <child link="camera_depth_frame" />
+    <child link="camera_link" />
   </joint>
 </robot>

Commit message: changed the formula for tf calculation

File: ajgar_description/urdf/ajgar.xacro (robot description, xacro)
@@ -174,5 +174,5 @@
   <child link="base_top"/>
   <axis xyz="-0.0 0.0 1.0"/>
-  <limit upper="2.879793" lower="-2.879793" effort="100" velocity="100" />
+  <limit upper="3.14159" lower="-3.14159" effort="100" velocity="100" />
 </joint>
 <joint name="shoulder_joint" type="revolute">
@@ -181,5 +181,5 @@
   <child link="shoulder"/>
   <axis xyz="-0.0 1.0 -0.0"/>
-  <limit upper="2.879793" lower="-2.879793" effort="100" velocity="100" />
+  <limit upper="2.16421" lower="-2.33874" effort="100" velocity="100" />
 </joint>
 <joint name="elbow_joint" type="revolute">
@@ -188,5 +188,5 @@
   <child link="elbow"/>
   <axis xyz="0.0 -1.0 0.0"/>
-  <limit upper="2.879793" lower="-2.879793" effort="100" velocity="100" />
+  <limit upper="2.79253" lower="-2.79253" effort="100" velocity="100" />
 </joint>
 <joint name="lower_wrist_joint" type="revolute">
@@ -195,5 +195,5 @@
   <child link="wrist"/>
   <axis xyz="0.0 0.0 1.0"/>
-    <limit upper="2.879793" lower="-2.879793" effort="100" velocity="100" />
+    <limit upper="3.14159" lower="-3.14159" effort="100" velocity="100" />
 </joint>
 <joint name="upper_wrist_joint" type="revolute">
@@ -202,5 +202,5 @@
   <child link="suction"/>
   <axis xyz="-0.0 1.0 -0.0"/>
-    <limit upper="2.879793" lower="-2.879793" effort="100" velocity="100" />
+    <limit upper="0.837758" lower="-2.58309" effort="100" velocity="100" />
 </joint>
 <joint name="end_joint" type="revolute">
@@ -209,5 +209,5 @@
   <child link="end"/>
   <axis xyz="-0.0 -0.0 -1.0"/>
-    <limit upper="2.879793" lower="-2.879793" effort="100" velocity="100" />
+    <limit upper="3.14159" lower="-3.14159" effort="100" velocity="100" />
 </joint>
 <joint name="kinect_joint" type="fixed">

Commit message: changed the formula for tf calculation

File: ajgar_description/urdf/ajgar.xacro (robot description, xacro)
@@ -145,23 +145,4 @@
   </collision>
 </link>
-<link name="camera_depth_frame">
-    <collision>
-      <origin xyz="0 0 0" rpy="1.57 0 0" />
-      <geometry>
-        <mesh filename="package://ur5_description/meshes/kinect.stl" scale="0.005 0.005 0.005" />
-      </geometry>
-    </collision>
-    <visual>
-      <origin xyz="0 0 0" rpy="1.57 -1.57 0" />
-      <geometry>
-        <mesh filename="package://ur5_description/meshes/kinect.stl" scale="0.005 0.005 0.005" />
-      </geometry>
-    </visual>
-    <inertial>
-      <mass value="1e-5" />
-      <origin xyz="0 0 0" rpy="0 0 0" />
-      <inertia ixx="1e-6" ixy="0" ixz="0" iyy="1e-6" iyz="0" izz="1e-6" />
-    </inertial>
-  </link>
 <joint name="world_joint" type="fixed">
     <parent link="world" />
@@ -174,5 +155,5 @@
   <child link="base_top"/>
   <axis xyz="-0.0 0.0 1.0"/>
-  <limit upper="2.879793" lower="-2.879793" effort="100" velocity="100" />
+  <limit upper="3.14159" lower="-3.14159" effort="100" velocity="100" />
 </joint>
 <joint name="shoulder_joint" type="revolute">
@@ -181,5 +162,5 @@
   <child link="shoulder"/>
   <axis xyz="-0.0 1.0 -0.0"/>
-  <limit upper="2.879793" lower="-2.879793" effort="100" velocity="100" />
+  <limit upper="2.16421" lower="-2.33874" effort="100" velocity="100" />
 </joint>
 <joint name="elbow_joint" type="revolute">
@@ -188,5 +169,5 @@
   <child link="elbow"/>
   <axis xyz="0.0 -1.0 0.0"/>
-  <limit upper="2.879793" lower="-2.879793" effort="100" velocity="100" />
+  <limit upper="2.79253" lower="-2.79253" effort="100" velocity="100" />
 </joint>
 <joint name="lower_wrist_joint" type="revolute">
@@ -195,5 +176,5 @@
   <child link="wrist"/>
   <axis xyz="0.0 0.0 1.0"/>
-    <limit upper="2.879793" lower="-2.879793" effort="100" velocity="100" />
+    <limit upper="3.14159" lower="-3.14159" effort="100" velocity="100" />
 </joint>
 <joint name="upper_wrist_joint" type="revolute">
@@ -202,5 +183,5 @@
   <child link="suction"/>
   <axis xyz="-0.0 1.0 -0.0"/>
-    <limit upper="2.879793" lower="-2.879793" effort="100" velocity="100" />
+    <limit upper="0.837758" lower="-2.58309" effort="100" velocity="100" />
 </joint>
 <joint name="end_joint" type="revolute">
@@ -209,10 +190,5 @@
   <child link="end"/>
   <axis xyz="-0.0 -0.0 -1.0"/>
-    <limit upper="2.879793" lower="-2.879793" effort="100" velocity="100" />
-</joint>
-<joint name="kinect_joint" type="fixed">
-  <origin xyz="0.612 -0.15 1.5" rpy="0 1.57 0" />
-  <parent link="base_link" />
-  <child link="camera_depth_frame" />
+    <limit upper="3.14159" lower="-3.14159" effort="100" velocity="100" />
 </joint>
 </robot>

Commit message: jc ganda aadmi hai

File: ajgar_description/urdf/ajgar.xacro (robot description, xacro)
@@ -144,4 +144,23 @@
     </geometry>
   </collision>
+</link>
+<link name="camera_depth_frame">
+  <collision>
+    <origin xyz="0 0 0" rpy="1.57 0 0" />
+    <geometry>
+      <mesh filename="package://ur5_description/meshes/kinect.stl" scale="0.005 0.005 0.005" />
+    </geometry>
+  </collision>
+  <visual>
+    <origin xyz="0 0 0" rpy="1.57 -1.57 0" />
+    <geometry>
+      <mesh filename="package://ur5_description/meshes/kinect.stl" scale="0.005 0.005 0.005" />
+    </geometry>
+  </visual>
+  <inertial>
+    <mass value="1e-5" />
+    <origin xyz="0 0 0" rpy="0 0 0" />
+    <inertia ixx="1e-6" ixy="0" ixz="0" iyy="1e-6" iyz="0" izz="1e-6" />
+  </inertial>
 </link>
 <link name="camera_link">

Commit message: modifed arm position wrt trolley

File: ajgar_description/urdf/ajgar.xacro (robot description, xacro)
@@ -1,4 +1,4 @@
 <?xml version="1.0" ?>
-<robot name="ajgar_description" xmlns:xacro="http://www.ros.org/wiki/xacro">
+<robot name="ajgar" xmlns:xacro="http://www.ros.org/wiki/xacro">
 <xacro:include filename="$(find ajgar_description)/urdf/materials.xacro" />
 <xacro:include filename="$(find ajgar_description)/urdf/ajgar.trans" />
@@ -231,5 +231,5 @@
 </joint>
 <joint name="kinect_joint" type="fixed">
-  <origin xyz="0.612 -0.15 1.5" rpy="0 1.57 0" />
+  <origin xyz="0.612 0.0 1.5" rpy="0 1.57 0" />
   <parent link="base_link" />
   <child link="camera_link" />

Commit message: new world generated

File: ajgar_description/urdf/ajgar.xacro (robot description, xacro)
@@ -145,5 +145,5 @@
   </collision>
 </link>
-<link name="camera_depth_frame">
+<link name="camera_link">
   <collision>
     <origin xyz="0 0 0" rpy="1.57 0 0" />
@@ -231,5 +231,5 @@
 </joint>
 <joint name="kinect_joint" type="fixed">
-  <origin xyz="0.612 0.0 1.5" rpy="0 1.57 0" />
+  <origin xyz="0.40 0.0 1.0" rpy="0 1.57 0" />
   <parent link="base_link" />
   <child link="camera_link" />

Commit message: Remove ur5 arm and dependent moveit configuration

File: ajgar_description/urdf/ajgar.xacro (robot description, xacro)
@@ -149,5 +149,5 @@
     <origin xyz="0 0 0" rpy="1.57 0 0" />
     <geometry>
-      <mesh filename="package://ur5_description/meshes/kinect.stl" scale="0.005 0.005 0.005" />
+      <mesh filename="package://ajgar_description/meshes/kinect.stl" scale="0.005 0.005 0.005" />
     </geometry>
   </collision>
@@ -155,5 +155,5 @@
     <origin xyz="0 0 0" rpy="1.57 -1.57 0" />
     <geometry>
-      <mesh filename="package://ur5_description/meshes/kinect.stl" scale="0.005 0.005 0.005" />
+      <mesh filename="package://ajgar_description/meshes/kinect.stl" scale="0.005 0.005 0.005" />
     </geometry>
   </visual>
